File: Hardware/raspi mockup.brd (EAGLE design)
At the start: 85 x 56 mm, 45 parts, among them J1 QWIIC, J2 AVR_SPI_PROG_3X2TESTPOINTS, J3 4DLCD-24-320X240, U2 ADMP401, U3 ADMP401, U4 WM8960, U5 ATTINY84

Commit message: updating footprints, running checklist
Parts:
- added FD1, FD2, FD3, FD4: FIDUCIAL1X2, SparkFun-Aesthetics:FIDUCIAL-1X2
- added LOGO4: OSHW-LOGOS, SparkFun-Aesthetics:OSHW-LOGO-S
- added R4: 10k, SparkFun-Resistors:0603
- J3: value 4DLCD-24-320X240 -> 2.4" TFT
- moved LS2 1.50 mm to (75.5, 27.0)
- moved U$1 0.91 mm to (67.0, 23.2)
- moved U$2 0.28 mm to (65.8, 20.2)
Connections:
- net 3.3V: now also R4.2
- net CS: now also R4.1
Routing:
- net 3.3V: track 193.8 -> 198.1 mm
- net N$6: track 19.0 -> 17.5 mm
- net CS: track 32.9 -> 34.2 mm, vias 0 -> 1
- net N$22: track 13.7 -> 14.3 mm
Other:
- board text added: "Units in mm"
Changed lines of the file:
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@@
 <setting verticaltext="up"/>
 </settings>
-<grid distance="1" unitdist="mm" unit="mm" style="lines" multiple="1" display="yes" altdistance="0.05" altunitdist="mm" altunit="mm"/>
+<grid distance="0.5" unitdist="mm" unit="mm" style="lines" multiple="1" display="yes" altdistance="0.05" altunitdist="mm" altunit="mm"/>
 <layers>
 <layer number="1" name="Top" color="4" fill="1" visible="yes" active="yes"/>
@@
 <layer number="45" name="Holes" color="7" fill="1" visible="no" active="yes"/>
 <layer number="46" name="Milling" color="3" fill="1" visible="no" active="yes"/>
-<layer number="47" name="Measures" color="7" fill="1" visible="no" active="yes"/>
+<layer number="47" name="Measures" color="7" fill="1" visible="yes" active="yes"/>
 <layer number="48" name="Document" color="7" fill="1" visible="no" active="yes"/>
 <layer number="49" name="Reference" color="7" fill="1" visible="no" active="yes"/>
@@
 <board>
 <plain>
-<wire x1="3" y1="0" x2="0" y2="3" width="0.1524" layer="20" curve="-90"/>
-<wire x1="0" y1="3" x2="0" y2="53" width="0.1524" layer="20"/>
-<wire x1="0" y1="53" x2="3" y2="56" width="0.1524" layer="20" curve="-90"/>
+<wire x1="3" y1="0" x2="0" y2="3" width="0.2032" layer="20" curve="-90"/>
+<wire x1="0" y1="3" x2="0" y2="53" width="0.2032" layer="20"/>
+<wire x1="0" y1="53" x2="3" y2="56" width="0.2032" layer="20" curve="-90"/>
 <wire x1="3" y1="56" x2="82" y2="56" width="0.2032" layer="20"/>
-<wire x1="82" y1="56" x2="85" y2="53" width="0.1524" layer="20" curve="-90"/>
-<wire x1="85" y1="53" x2="85" y2="3" width="0.1524" layer="20"/>
-<wire x1="85" y1="3" x2="82" y2="0" width="0.1524" layer="20" curve="-90"/>
-<wire x1="82" y1="0" x2="3" y2="0" width="0.1524" layer="20"/>
+<wire x1="82" y1="56" x2="85" y2="53" width="0.2032" layer="20" curve="-90"/>
+<wire x1="85" y1="53" x2="85" y2="3" width="0.2032" layer="20"/>
+<wire x1="85" y1="3" x2="82" y2="0" width="0.2032" layer="20" curve="-90"/>
+<wire x1="82" y1="0" x2="3" y2="0" width="0.2032" layer="20"/>
 <wire x1="60.26" y1="49" x2="0" y2="49" width="0.1524" layer="51"/>
-<wire x1="0" y1="49" x2="0" y2="7" width="0.1524" layer="51"/>
+<wire x1="0" y1="49" x2="0" y2="7" width="0.2032" layer="51"/>
 <wire x1="0" y1="7" x2="60.26" y2="7" width="0.1524" layer="51"/>
 <wire x1="60.26" y1="7" x2="60.26" y2="49" width="0.1524" layer="51"/>
 <text x="46" y="-11" size="1.778" layer="51" font="vector">Andy England</text>
 <text x="84.6" y="9" size="1.778" layer="16" font="vector" ratio="15" rot="SMR270">v01</text>
+<dimension x1="3.5" y1="3.5" x2="0" y2="3.5" x3="1.75" y3="-3" textsize="1.778" layer="47"/>
+<dimension x1="0" y1="56" x2="0" y2="0" x3="-3.5" y3="28" textsize="1.778" layer="47"/>
+<dimension x1="0" y1="0" x2="85" y2="0" x3="42.5" y3="-4" textsize="1.778" layer="47"/>
+<dimension x1="61.5" y1="3.5" x2="85" y2="3.5" x3="73.25" y3="-2" textsize="1.778" layer="47"/>
+<dimension x1="61.5" y1="3.5" x2="61.5" y2="0" x3="-6.5" y3="1.75" textsize="1.778" layer="47"/>
+<dimension x1="61.5" y1="52.5" x2="61.5" y2="56" x3="-6.5" y3="54.25" textsize="1.778" layer="47"/>
+<dimension x1="3.5" y1="52.5" x2="0" y2="52.5" x3="1.75" y3="58.5" textsize="1.778" layer="47"/>
+<text x="-1" y="21.5" size="1.778" layer="47" font="vector" rot="R90">Units in mm</text>
 </plain>
 <attributes>
@@
 <attribute name="VALUE" x="10" y="6.294" size="0.6096" layer="27" font="vector" ratio="20" rot="R180" align="top-center"/>
 </element>
-<element name="LS2" library="SparkFun-Electromechanical" package="CVS-1508_PCBSPKR" value="CVS-1508" x="77" y="27" smashed="yes" rot="R270">
-<attribute name="PROD_ID" value="COM-14823" x="77" y="27" size="1.778" layer="27" rot="R270" display="off"/>
-<attribute name="VALUE" value="CVS-1508" x="77" y="27" size="1.778" layer="27" rot="R270" display="off"/>
-</element>
-<element name="J3" library="SparkFun-Displays" package="FPC05040-17204" value="4DLCD-24-320X240" x="20" y="27" smashed="yes" rot="MR90"/>
-<element name="U$2" library="buzzard_labels (14)" package="MACHINE_LEARNING0" value="" x="66" y="20" smashed="yes" rot="R90"/>
-<element name="U$1" library="buzzard_labels (14)" package="TOPHAT1" value="" x="67.95" y="23.15" smashed="yes" rot="R90"/>
+<element name="LS2" library="SparkFun-Electromechanical" package="CVS-1508_PCBSPKR" value="CVS-1508" x="75.5" y="27" smashed="yes" rot="R270">
+<attribute name="PROD_ID" value="COM-14823" x="75.5" y="27" size="1.778" layer="27" rot="R270" display="off"/>
+<attribute name="VALUE" value="CVS-1508" x="75.5" y="27" size="1.778" layer="27" rot="R270" display="off"/>
+</element>
+<element name="J3" library="SparkFun-Displays" package="FPC05040-17204" value="2.4&quot; TFT" x="20" y="27" smashed="yes" rot="MR90">
+<attribute name="PROD_ID" value="LCD-16014" x="20" y="27" size="1.778" layer="28" rot="MR90" display="off"/>
+<attribute name="VALUE" value="2.4&quot; TFT" x="20" y="27" size="1.778" layer="28" rot="MR90" display="off"/>
+</element>
+<element name="U$2" library="buzzard_labels (14)" package="MACHINE_LEARNING0" value="" x="65.8" y="20.2" smashed="yes" rot="R90"/>
+<element name="U$1" library="buzzard_labels (14)" package="TOPHAT1" value="" x="67.05" y="23.25" smashed="yes" rot="R90"/>
 <element name="LOGO1" library="SparkFun-Aesthetics" package="SFE_LOGO_NAME_FLAME_.1" value="SFE_LOGO_NAME_FLAME.1_INCH" x="64" y="27" smashed="yes" rot="R90"/>
 <element name="LOGO2" library="SparkFun-Aesthetics" package="SFE_LOGO_NAME_FLAME_.4" value="SFE_LOGO_NAME_FLAME.4_INCH" x="67" y="21" smashed="yes" rot="MR0"/>
 <element name="U$3" library="buzzard_labels (13)" package="MACHINE_LEARNING_TOPHAT0" value="" x="52" y="23" smashed="yes" rot="MR0"/>
 <element name="LOGO3" library="SparkFun-Aesthetics" package="QWIIC_4MM" value="QWIIC_LOGO_4MM" x="78.5" y="7" smashed="yes"/>
+<element name="LOGO4" library="SparkFun-Aesthetics" package="OSHW-LOGO-S" value="OSHW-LOGOS" x="83.5" y="27" smashed="yes" rot="MR270"/>
+<element name="FD1" library="SparkFun-Aesthetics" package="FIDUCIAL-1X2" value="FIDUCIAL1X2" x="2" y="9" smashed="yes"/>
+<element name="FD2" library="SparkFun-Aesthetics" package="FIDUCIAL-1X2" value="FIDUCIAL1X2" x="2" y="9" smashed="yes" rot="MR0"/>
+<element name="FD3" library="SparkFun-Aesthetics" package="FIDUCIAL-1X2" value="FIDUCIAL1X2" x="82" y="53" smashed="yes"/>
+<element name="FD4" library="SparkFun-Aesthetics" package="FIDUCIAL-1X2" value="FIDUCIAL1X2" x="82" y="53" smashed="yes" rot="MR0"/>
+<element name="R4" library="SparkFun-Resistors" package="0603" value="10k" x="37.55" y="52.5" smashed="yes" rot="R270">
+<attribute name="NAME" x="38.312" y="52.5" size="0.6096" layer="25" font="vector" ratio="20" rot="R270" align="bottom-center"/>
+<attribute name="PROD_ID" value="RES-00824" x="37.55" y="52.5" size="1.778" layer="27" rot="R270" display="off"/>
+<attribute name="VALUE" x="36.788" y="52.5" size="0.6096" layer="27" font="vector" ratio="20" rot="R270" align="top-center"/>
+</element>
 </elements>
 <signals>
@@
 <via x="47" y="44" extent="1-16" drill="0.381"/>
 <wire x1="47" y1="44" x2="43.7" y2="47.3" width="0.1778" layer="1"/>
-<wire x1="43.7" y1="47.3" x2="28.7" y2="47.3" width="0.1778" layer="1"/>
+<wire x1="43.7" y1="47.3" x2="37.55" y2="47.3" width="0.1778" layer="1"/>
 <via x="28.7" y="47.3" extent="1-16" drill="0.381"/>
+<wire x1="37.55" y1="47.3" x2="28.7" y2="47.3" width="0.1778" layer="1"/>
 <wire x1="28.7" y1="47.3" x2="28.69" y2="47.31" width="0.1778" layer="16"/>
 <wire x1="28.69" y1="47.31" x2="28.69" y2="49.585" width="0.1778" layer="16"/>
@@
 <wire x1="70.25" y1="45.75" x2="70" y2="45.75" width="0.1778" layer="1"/>
 <wire x1="70.25" y1="44.8" x2="70.25" y2="45.75" width="0.1778" layer="1"/>
+<contactref element="R4" pad="2"/>
+<wire x1="37.55" y1="51.65" x2="37.55" y2="47.3" width="0.1778" layer="1"/>
 </signal>
 <signal name="GND">
@@
 <contactref element="LS2" pad="-"/>
 <wire x1="73.8" y1="29.05" x2="73.8" y2="38.95" width="0.1778" layer="1"/>
-<wire x1="73.2" y1="27" x2="73.2" y2="28.45" width="0.1778" layer="1"/>
-<wire x1="73.2" y1="28.45" x2="73.8" y2="29.05" width="0.1778" layer="1"/>
+<wire x1="71.7" y1="27" x2="71.75" y2="27" width="0.1778" layer="1"/>
+<wire x1="71.75" y1="27" x2="73.8" y2="29.05" width="0.1778" layer="1"/>
 </signal>
 <signal name="N$6">
@@
 <wire x1="74.3" y1="40.75" x2="74.3" y2="29.05" width="0.1778" layer="1"/>
 <contactref element="LS2" pad="+"/>
-<wire x1="76.35" y1="27" x2="80.8" y2="27" width="0.1778" layer="1"/>
+<wire x1="76.35" y1="27" x2="79.3" y2="27" width="0.1778" layer="1"/>
 <wire x1="74.3" y1="29.05" x2="76.35" y2="27" width="0.1778" layer="1"/>
 </signal>
@@
 <wire x1="37.55" y1="45.55" x2="37.55" y2="54.65" width="0.1778" layer="16"/>
 <wire x1="37.55" y1="54.65" x2="36.885" y2="55.315" width="0.1778" layer="16"/>
+<contactref element="R4" pad="1"/>
+<wire x1="37.55" y1="53.35" x2="37.55" y2="54.65" width="0.1778" layer="1"/>
+<via x="37.55" y="54.65" extent="1-16" drill="0.381"/>
 </signal>
 <signal name="D/C">

Commit message: post review changes
Parts:
- added J4: (no value), SparkFun-Connectors:1X02_NO_SILK
- added JP1: JUMPER-SMT_2_NC_TRACE_NO-SILK, SparkFun-Jumpers:SMT-JUMPER_2_NC_TRACE_NO-SILK
- added TP1: TEST-POINT3X4, SparkFun-Connectors:PAD.03X.04
- added U$4: (no value), buzzard_labels (16):02
- added U$5: (no value), buzzard_labels (16):53
- added U$6: (no value), buzzard_labels (16):A0
- added U$7: (no value), buzzard_labels (16):B1
- added U$8: (no value), buzzard_labels (17):I2C3
- moved FD3 2.54 mm to (79.5, 53.0)
- moved FD4 2.54 mm to (79.5, 53.0)
Connections:
- net !RESET renamed !RST_SCREEN
- net !RST renamed !RST_ATTINY
- net CS renamed !CS
- net INT renamed !INT
- removed net N$31: J1.3, R2.1, U1.5
- removed net N$32: J1.4, R3.1, U1.3
- new net N$10: TP1.P$1, U4.30
- new net N$4: J3.8, JP1.1
- new net N$5: J4.1, U4.19
- new net N$7: J4.2, U4.22
- net 3.3V: now also JP1.2; no longer J3.8
- net SCL: now also J1.3, R2.1, U1.5
- net SDA: now also J1.4, R3.1, U1.3
Routing:
- net SDA: track 36.9 -> 171.7 mm, vias 1 -> 6
- net SCL: track 37.5 -> 167.9 mm, vias 1 -> 4
- net N$32: track 103.7 -> 0.00 mm, vias 3 -> 0
- net N$31: track 98.4 -> 0.00 mm, vias 3 -> 0
- net N$7: track 0.00 -> 21.5 mm, vias 0 -> 1
- net N$5: track 0.00 -> 19.3 mm, vias 0 -> 1
- net 3.3V: track 198.1 -> 203.5 mm, vias 6 -> 8
- net N$4: track 0.00 -> 2.40 mm
- net N$10: track 0.00 -> 2.39 mm
- net BTN_LEFT: track 18.1 -> 18.7 mm
