File: Hardware/raspi mockup.brd (EAGLE design)
At the start: 85 x 56 mm, 59 parts, among them J1 QWIIC, J2 AVR_SPI_PROG_3X2TESTPOINTS, J3 2.4" TFT, U2 ADMP401, U3 ADMP401, U4 WM8960, U5 ATTINY84

Commit message: pre design review for REDs
Parts:
- removed J4: (no value), SparkFun-Connectors:1X02_NO_SILK
- removed TP1: TEST-POINT3X4, SparkFun-Connectors:PAD.03X.04
- removed U$3: (no value), buzzard_labels (13):MACHINE_LEARNING_TOPHAT0
- added C13: 10nF, SparkFun-Capacitors:0603
- added Q1: 220mA/50V/3.5Ω, SparkFun-DiscreteSemi:SOT23-3
- added Y1: 24 MHz, SparkFun-Clocks:RESONATOR-SMD-3.2X2.5
- U$1: device buzzard_labels (14):TOPHAT1 -> buzzard_labels (21):_TOP_PHAT1
- U$2: device buzzard_labels (14):MACHINE_LEARNING0 -> buzzard_labels (21):TOP_PHAT0
- moved U$2 16.4 mm to (82.0, 22.8)
- moved LOGO1 15.5 mm to (79.5, 27.0)
- moved U$1 13.1 mm to (54.0, 22.0), flipped to the bottom, turned to 0 degrees
- moved LS2 7.52 mm to (68.0, 26.5), turned to 180 degrees
- moved C5 5.02 mm to (66.5, 47.5), turned to 0 degrees
- moved C8 3.16 mm to (77.5, 39.5), turned to 90 degrees
- moved J3 1.90 mm to (20.0, 28.9)
- moved JP1 1.90 mm to (22.9, 23.5)
- moved R3 1.55 mm to (72.5, 3.00)
- moved R2 1.50 mm to (72.5, 1.50)
- moved C7 0.71 mm to (76.0, 39.5), turned to 90 degrees
- moved C6 0.50 mm to (72.0, 37.5)
- turned C4 to 180 degrees
Connections:
- removed net ADC-LRC: U4.15
- removed net N$10: TP1.P$1, U4.30
- removed net N$5: J4.1, U4.19
- removed net N$7: J4.2, U4.22
- new net N$11: U4.11, Y1.3
- net 3.3V: now also C13.1, Y1.1, Y1.4
- net DAC-LRC: now also U4.15
- net GND: now also C13.2, Y1.2
- net SCL: now also J1.4; no longer J1.3
- net SDA: now also J1.3; no longer J1.4
Routing:
- net N$7: track 21.5 -> 0.00 mm, vias 1 -> 0
- net N$5: track 19.3 -> 0.00 mm, vias 1 -> 0
- net GND: track 15.1 -> 6.11 mm, vias 37 -> 40
- net N$6: track 17.5 -> 21.1 mm
- net N$16: track 2.07 -> 4.80 mm
- net N$11: track 0.00 -> 2.46 mm
- net N$10: track 2.39 -> 0.00 mm
- net N$38: track 1.66 -> 4.04 mm
- net DAC-LRC: track 25.5 -> 27.8 mm, vias 1 -> 3
- net 3.3V: track 203.5 -> 201.2 mm
- net SDO: track 31.1 -> 29.2 mm
- net !CS: track 34.2 -> 32.3 mm
- net SDI: track 20.5 -> 18.6 mm
- net SCK: track 25.0 -> 23.1 mm
- net !RST_SCREEN: track 32.7 -> 30.8 mm
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