File: Hardware/raspi mockup.sch (EAGLE design)
At the start: 42 parts, among them J1 QWIIC, J2 AVR_SPI_PROG_3X2TESTPOINTS, J3 4DLCD-24-320X240, U1 RASPBERRY_PI_40BTM-NOHOLES, U2 ADMP401, U3 ADMP401, U4 WM8960, U5 ATTINY84

Commit message: updating int pin
Connections:
- net INT: now also U1.D25
Changed lines of the file:
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@@
 <label x="233.68" y="99.06" size="1.27" layer="95" font="vector" xref="yes"/>
+</segment>
+<segment>
+<pinref part="U1" gate="U1" pin="D25"/>
+<wire x1="40.64" y1="93.98" x2="43.18" y2="93.98" width="0.1524" layer="91"/>
+<label x="43.18" y="93.98" size="1.27" layer="95" xref="yes"/>
 </segment>
 </net>

Commit message: updating footprints, running checklist
Parts:
- added FD1, FD2, FD3, FD4: FIDUCIAL1X2, SparkFun-Aesthetics:FIDUCIAL1X2
- added LOGO4: OSHW-LOGOS, SparkFun-Aesthetics:OSHW-LOGOS
- added R4: 10k, SparkFun-Resistors:10KOHM-0603-1/10W-1%
- J3: value 4DLCD-24-320X240 -> 2.4" TFT
Connections:
- net 3.3V: now also R4.2
- net CS: now also R4.1
Other:
- note added: "Cut I2C Jumper to remove pullup jumpers from the I2C bus."
- moved on the sheet: J3
Changed lines of the file:
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@@
 <part name="SUPPLY8" library="SparkFun-PowerSymbols" deviceset="5V" device=""/>
 <part name="LS2" library="SparkFun-Electromechanical" deviceset="SPEAKER" device="CVS-1508" value="CVS-1508"/>
-<part name="J3" library="SparkFun-Displays" deviceset="4DLCD-24-320X240" device=""/>
+<part name="J3" library="SparkFun-Displays" deviceset="4DLCD-24-320X240" device="" value="2.4&quot; TFT"/>
 <part name="SUPPLY11" library="SparkFun-PowerSymbols" deviceset="3.3V" device=""/>
 <part name="GND9" library="SparkFun-PowerSymbols" deviceset="GND" device=""/>
@@
 <part name="LOGO2" library="SparkFun-Aesthetics" deviceset="SFE_LOGO_NAME_FLAME" device=".4_INCH"/>
 <part name="LOGO3" library="SparkFun-Aesthetics" deviceset="QWIIC_LOGO" device="_4MM"/>
+<part name="LOGO4" library="SparkFun-Aesthetics" deviceset="OSHW-LOGO" device="S"/>
+<part name="FD1" library="SparkFun-Aesthetics" deviceset="FIDUCIAL" device="1X2"/>
+<part name="FD2" library="SparkFun-Aesthetics" deviceset="FIDUCIAL" device="1X2"/>
+<part name="FD3" library="SparkFun-Aesthetics" deviceset="FIDUCIAL" device="1X2"/>
+<part name="FD4" library="SparkFun-Aesthetics" deviceset="FIDUCIAL" device="1X2"/>
+<part name="R4" library="SparkFun-Resistors" deviceset="10KOHM" device="-0603-1/10W-1%" value="10k"/>
+<part name="SUPPLY12" library="SparkFun-PowerSymbols" deviceset="3.3V" device=""/>
 </parts>
 <sheets>
@@
 <text x="129.54" y="127" size="2.54" layer="97" font="vector">ATTiny Button Master</text>
 <text x="129.54" y="180.34" size="2.54" layer="97" font="vector">WS2812 LED's</text>
+<text x="25.4" y="167.64" size="1.778" layer="97" font="vector">Cut I2C Jumper to
+remove pullup jumpers
+from the I2C bus.</text>
 </plain>
 <instances>
@@
 <attribute name="VALUE" x="119.38" y="27.686" size="1.27" layer="96" font="vector" rot="R180"/>
 </instance>
-<instance part="J3" gate="G$1" x="96.52" y="104.14" smashed="yes">
-<attribute name="NAME" x="86.36" y="114.808" size="1.778" layer="95" font="vector"/>
-<attribute name="VALUE" x="86.36" y="93.98" size="1.778" layer="96" font="vector"/>
-</instance>
-<instance part="SUPPLY11" gate="G$1" x="81.28" y="114.3" smashed="yes" rot="MR0">
-<attribute name="VALUE" x="81.28" y="117.094" size="1.778" layer="96" rot="MR0" align="bottom-center"/>
-</instance>
-<instance part="GND9" gate="1" x="78.74" y="93.98" smashed="yes" rot="MR0">
-<attribute name="VALUE" x="78.74" y="93.726" size="1.778" layer="96" rot="MR0" align="top-center"/>
+<instance part="J3" gate="G$1" x="91.44" y="104.14" smashed="yes">
+<attribute name="NAME" x="81.28" y="114.808" size="1.778" layer="95" font="vector"/>
+<attribute name="VALUE" x="81.28" y="93.98" size="1.778" layer="96" font="vector"/>
+</instance>
+<instance part="SUPPLY11" gate="G$1" x="76.2" y="114.3" smashed="yes" rot="MR0">
+<attribute name="VALUE" x="76.2" y="117.094" size="1.778" layer="96" rot="MR0" align="bottom-center"/>
+</instance>
+<instance part="GND9" gate="1" x="73.66" y="93.98" smashed="yes" rot="MR0">
+<attribute name="VALUE" x="73.66" y="93.726" size="1.778" layer="96" rot="MR0" align="top-center"/>
 </instance>
 <instance part="LOGO1" gate="G$1" x="68.58" y="157.48" smashed="yes"/>
 <instance part="LOGO2" gate="G$1" x="68.58" y="157.48" smashed="yes"/>
 <instance part="LOGO3" gate="G$1" x="96.52" y="157.48" smashed="yes"/>
+<instance part="LOGO4" gate="G$1" x="96.52" y="147.32" smashed="yes"/>
+<instance part="FD1" gate="G$1" x="238.76" y="30.48" smashed="yes"/>
+<instance part="FD2" gate="G$1" x="236.22" y="30.48" smashed="yes"/>
+<instance part="FD3" gate="G$1" x="236.22" y="27.94" smashed="yes"/>
+<instance part="FD4" gate="G$1" x="238.76" y="27.94" smashed="yes"/>
+<instance part="R4" gate="G$1" x="119.38" y="111.76" smashed="yes" rot="R90">
+<attribute name="NAME" x="117.856" y="111.76" size="1.778" layer="95" font="vector" rot="R90" align="bottom-center"/>
+<attribute name="VALUE" x="120.904" y="111.76" size="1.778" layer="96" font="vector" rot="R90" align="top-center"/>
+</instance>
+<instance part="SUPPLY12" gate="G$1" x="119.38" y="119.38" smashed="yes" rot="MR0">
+<attribute name="VALUE" x="119.38" y="122.174" size="1.778" layer="96" rot="MR0" align="bottom-center"/>
+</instance>
 </instances>
 <busses>
@@
 <segment>
 <pinref part="SUPPLY11" gate="G$1" pin="3.3V"/>
-<wire x1="81.28" y1="114.3" x2="81.28" y2="111.76" width="0.1524" layer="91"/>
+<wire x1="76.2" y1="114.3" x2="76.2" y2="111.76" width="0.1524" layer="91"/>
 <pinref part="J3" gate="G$1" pin="VCC"/>
-<wire x1="81.28" y1="111.76" x2="83.82" y2="111.76" width="0.1524" layer="91"/>
+<wire x1="76.2" y1="111.76" x2="78.74" y2="111.76" width="0.1524" layer="91"/>
 <pinref part="J3" gate="G$1" pin="LEDA"/>
-<wire x1="83.82" y1="104.14" x2="81.28" y2="104.14" width="0.1524" layer="91"/>
-<wire x1="81.28" y1="104.14" x2="81.28" y2="111.76" width="0.1524" layer="91"/>
-<junction x="81.28" y="111.76"/>
+<wire x1="78.74" y1="104.14" x2="76.2" y2="104.14" width="0.1524" layer="91"/>
+<wire x1="76.2" y1="104.14" x2="76.2" y2="111.76" width="0.1524" layer="91"/>
+<junction x="76.2" y="111.76"/>
+</segment>
+<segment>
+<pinref part="SUPPLY12" gate="G$1" pin="3.3V"/>
+<pinref part="R4" gate="G$1" pin="2"/>
+<wire x1="119.38" y1="119.38" x2="119.38" y2="116.84" width="0.1524" layer="91"/>
 </segment>
 </net>
@@
 <segment>
 <pinref part="J3" gate="G$1" pin="LEDK"/>
-<wire x1="83.82" y1="106.68" x2="78.74" y2="106.68" width="0.1524" layer="91"/>
+<wire x1="78.74" y1="106.68" x2="73.66" y2="106.68" width="0.1524" layer="91"/>
 <pinref part="J3" gate="G$1" pin="GND"/>
-<wire x1="78.74" y1="106.68" x2="78.74" y2="99.06" width="0.1524" layer="91"/>
-<wire x1="78.74" y1="99.06" x2="83.82" y2="99.06" width="0.1524" layer="91"/>
-<wire x1="78.74" y1="99.06" x2="78.74" y2="96.52" width="0.1524" layer="91"/>
-<junction x="78.74" y="99.06"/>
+<wire x1="73.66" y1="106.68" x2="73.66" y2="99.06" width="0.1524" layer="91"/>
+<wire x1="73.66" y1="99.06" x2="78.74" y2="99.06" width="0.1524" layer="91"/>
+<wire x1="73.66" y1="99.06" x2="73.66" y2="96.52" width="0.1524" layer="91"/>
+<junction x="73.66" y="99.06"/>
 <pinref part="GND9" gate="1" pin="GND"/>
 </segment>
@@
 <segment>
 <pinref part="J3" gate="G$1" pin="SCK"/>
-<wire x1="109.22" y1="106.68" x2="111.76" y2="106.68" width="0.1524" layer="91"/>
-<label x="111.76" y="106.68" size="1.27" layer="95" xref="yes"/>
+<wire x1="104.14" y1="106.68" x2="106.68" y2="106.68" width="0.1524" layer="91"/>
+<label x="106.68" y="106.68" size="1.27" layer="95" xref="yes"/>
 </segment>
 <segment>
@@
 <segment>
 <pinref part="J3" gate="G$1" pin="CS"/>
-<wire x1="109.22" y1="104.14" x2="111.76" y2="104.14" width="0.1524" layer="91"/>
-<label x="111.76" y="104.14" size="1.27" layer="95" xref="yes"/>
+<wire x1="104.14" y1="104.14" x2="119.38" y2="104.14" width="0.1524" layer="91"/>
+<label x="121.92" y="104.14" size="1.27" layer="95" xref="yes"/>
+<pinref part="R4" gate="G$1" pin="1"/>
+<wire x1="119.38" y1="104.14" x2="121.92" y2="104.14" width="0.1524" layer="91"/>
+<wire x1="119.38" y1="106.68" x2="119.38" y2="104.14" width="0.1524" layer="91"/>
+<junction x="119.38" y="104.14"/>
 </segment>
 <segment>
@@
 <segment>
 <pinref part="J3" gate="G$1" pin="D/C"/>
-<wire x1="109.22" y1="101.6" x2="111.76" y2="101.6" width="0.1524" layer="91"/>
-<label x="111.76" y="101.6" size="1.27" layer="95" xref="yes"/>
+<wire x1="104.14" y1="101.6" x2="106.68" y2="101.6" width="0.1524" layer="91"/>
+<label x="106.68" y="101.6" size="1.27" layer="95" xref="yes"/>
 </segment>
 <segment>
@@
 <segment>
 <pinref part="J3" gate="G$1" pin="SDI"/>
-<wire x1="109.22" y1="111.76" x2="111.76" y2="111.76" width="0.1524" layer="91"/>
-<label x="111.76" y="111.76" size="1.27" layer="95" xref="yes"/>
+<wire x1="104.14" y1="111.76" x2="106.68" y2="111.76" width="0.1524" layer="91"/>
+<label x="106.68" y="111.76" size="1.27" layer="95" xref="yes"/>
 </segment>
 <segment>
@@
 <segment>
 <pinref part="J3" gate="G$1" pin="SDO"/>
-<wire x1="109.22" y1="99.06" x2="111.76" y2="99.06" width="0.1524" layer="91"/>
-<label x="111.76" y="99.06" size="1.27" layer="95" xref="yes"/>
+<wire x1="104.14" y1="99.06" x2="106.68" y2="99.06" width="0.1524" layer="91"/>
+<label x="106.68" y="99.06" size="1.27" layer="95" xref="yes"/>
 </segment>
 <segment>
@@
 <segment>
 <pinref part="J3" gate="G$1" pin="RESET"/>
-<wire x1="109.22" y1="109.22" x2="111.76" y2="109.22" width="0.1524" layer="91"/>
-<label x="111.76" y="109.22" size="1.27" layer="95" xref="yes"/>
+<wire x1="104.14" y1="109.22" x2="106.68" y2="109.22" width="0.1524" layer="91"/>
+<label x="106.68" y="109.22" size="1.27" layer="95" xref="yes"/>
 </segment>
 <segment>
@@
 </drawing>
 <compatibility>
+<note version="6.3" minversion="6.2.2" severity="warning">
+Since Version 6.2.2 text objects can contain more than one line,
+which will not be processed correctly with this version.
+</note>
 <note version="8.3" severity="warning">
 Since Version 8.3, EAGLE supports URNs for individual library

Commit message: post review changes
Parts:
- added J4: (no value), SparkFun-Connectors:CONN_021X02_NO_SILK
- added JP1: JUMPER-SMT_2_NC_TRACE_NO-SILK, SparkFun-Jumpers:JUMPER-SMT_2_NC_TRACE_NO-SILK
- added TP1: TEST-POINT3X4, SparkFun-Connectors:TEST-POINT3X4
Connections:
- net !RESET renamed !RST_SCREEN
- net !RST renamed !RST_ATTINY
- net CS renamed !CS
- net INT renamed !INT
- removed net N$31: J1.3, R2.1, U1.SCL/D3
- removed net N$32: J1.4, R3.1, U1.SDA/D2
- new net N$10: TP1.1, U4.MONO_OUT
- new net N$4: J3.LEDA, JP1.1
- new net N$5: J4.1, U4.SPEAKER_RN
- new net N$7: J4.2, U4.SPEAKER_RP
- net 3.3V: now also JP1.2; no longer J3.LEDA
- net SCL: now also J1.3, R2.1, U1.SCL/D3
- net SDA: now also J1.4, R3.1, U1.SDA/D2
Other:
- note added: "7-bit Unshifted I2C Address: 0x34"
Changed lines of the file:
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@@
 <part name="R4" library="SparkFun-Resistors" deviceset="10KOHM" device="-0603-1/10W-1%" value="10k"/>
 <part name="SUPPLY12" library="SparkFun-PowerSymbols" deviceset="3.3V" device=""/>
+<part name="JP1" library="SparkFun-Jumpers" deviceset="JUMPER-SMT_2_NC_TRACE" device="_NO-SILK" package3d_urn="urn:adsk.eagle:package:39286/1"/>
+<part name="J4" library="SparkFun-Connectors" deviceset="CONN_02" device="1X02_NO_SILK"/>
+<part name="TP1" library="SparkFun-Connectors" deviceset="TEST-POINT" device="3X4" value="TEST-POINT3X4"/>
 </parts>
 <sheets>
@@
 remove pullup jumpers
 from the I2C bus.</text>
+<text x="198.12" y="73.66" size="1.27" layer="97" font="vector">7-bit Unshifted I2C Address: 0x34</text>
 </plain>
 <instances>
@@
 <attribute name="VALUE" x="81.28" y="93.98" size="1.778" layer="96" font="vector"/>
 </instance>
-<instance part="SUPPLY11" gate="G$1" x="76.2" y="114.3" smashed="yes" rot="MR0">
-<attribute name="VALUE" x="76.2" y="117.094" size="1.778" layer="96" rot="MR0" align="bottom-center"/>
+<instance part="SUPPLY11" gate="G$1" x="76.2" y="119.38" smashed="yes" rot="MR0">
+<attribute name="VALUE" x="76.2" y="122.174" size="1.778" layer="96" rot="MR0" align="bottom-center"/>
 </instance>
 <instance part="GND9" gate="1" x="73.66" y="93.98" smashed="yes" rot="MR0">
@@
 <instance part="SUPPLY12" gate="G$1" x="119.38" y="119.38" smashed="yes" rot="MR0">
 <attribute name="VALUE" x="119.38" y="122.174" size="1.778" layer="96" rot="MR0" align="bottom-center"/>
+</instance>
+<instance part="JP1" gate="G$1" x="71.12" y="111.76" smashed="yes" rot="R90">
+<attribute name="NAME" x="68.58" y="109.22" size="1.778" layer="95" font="vector" rot="R90"/>
+<attribute name="VALUE" x="73.66" y="109.22" size="1.778" layer="96" font="vector" rot="R90" align="top-left"/>
+</instance>
+<instance part="J4" gate="G$1" x="99.06" y="38.1" smashed="yes" rot="MR0">
+<attribute name="VALUE" x="101.6" y="33.274" size="1.778" layer="96" font="vector" rot="MR0"/>
+<attribute name="NAME" x="101.6" y="43.688" size="1.778" layer="95" font="vector" rot="MR0"/>
+</instance>
+<instance part="TP1" gate="G$1" x="91.44" y="45.72" smashed="yes">
+<attribute name="NAME" x="88.9" y="48.26" size="1.778" layer="95" font="vector"/>
+<attribute name="VALUE" x="88.9" y="43.18" size="1.778" layer="96" font="vector"/>
 </instance>
 </instances>
@@
 <segment>
 <pinref part="SUPPLY11" gate="G$1" pin="3.3V"/>
-<wire x1="76.2" y1="114.3" x2="76.2" y2="111.76" width="0.1524" layer="91"/>
+<wire x1="76.2" y1="119.38" x2="76.2" y2="116.84" width="0.1524" layer="91"/>
 <pinref part="J3" gate="G$1" pin="VCC"/>
+<wire x1="76.2" y1="116.84" x2="76.2" y2="111.76" width="0.1524" layer="91"/>
 <wire x1="76.2" y1="111.76" x2="78.74" y2="111.76" width="0.1524" layer="91"/>
-<pinref part="J3" gate="G$1" pin="LEDA"/>
-<wire x1="78.74" y1="104.14" x2="76.2" y2="104.14" width="0.1524" layer="91"/>
-<wire x1="76.2" y1="104.14" x2="76.2" y2="111.76" width="0.1524" layer="91"/>
-<junction x="76.2" y="111.76"/>
+<pinref part="JP1" gate="G$1" pin="2"/>
+<wire x1="76.2" y1="116.84" x2="71.12" y2="116.84" width="0.1524" layer="91"/>
+<junction x="76.2" y="116.84"/>
 </segment>
 <segment>
@@
 <label x="233.68" y="91.44" size="1.27" layer="95" font="vector" xref="yes"/>
 </segment>
+<segment>
+<pinref part="J1" gate="G$1" pin="3"/>
+<pinref part="U1" gate="U1" pin="SCL/D3"/>
+<wire x1="68.58" y1="149.86" x2="53.34" y2="149.86" width="0.1524" layer="91"/>
+<pinref part="R2" gate="G$1" pin="1"/>
+<wire x1="53.34" y1="149.86" x2="45.72" y2="149.86" width="0.1524" layer="91"/>
+<wire x1="45.72" y1="149.86" x2="40.64" y2="149.86" width="0.1524" layer="91"/>
+<wire x1="45.72" y1="154.94" x2="45.72" y2="149.86" width="0.1524" layer="91"/>
+<junction x="45.72" y="149.86"/>
+<wire x1="53.34" y1="149.86" x2="53.34" y2="147.32" width="0.1524" layer="91"/>
+<junction x="53.34" y="149.86"/>
+<wire x1="53.34" y1="147.32" x2="55.88" y2="147.32" width="0.1524" layer="91"/>
+<label x="55.88" y="147.32" size="1.27" layer="95" xref="yes"/>
+</segment>
 </net>
 <net name="SDA" class="0">
@@
 <wire x1="231.14" y1="96.52" x2="233.68" y2="96.52" width="0.1524" layer="91"/>
 <label x="233.68" y="96.52" size="1.27" layer="95" font="vector" xref="yes"/>
+</segment>
+<segment>
+<pinref part="U1" gate="U1" pin="SDA/D2"/>
+<pinref part="J1" gate="G$1" pin="4"/>
+<wire x1="40.64" y1="152.4" x2="50.8" y2="152.4" width="0.1524" layer="91"/>
+<pinref part="R3" gate="G$1" pin="1"/>
+<wire x1="50.8" y1="152.4" x2="60.96" y2="152.4" width="0.1524" layer="91"/>
+<wire x1="60.96" y1="152.4" x2="68.58" y2="152.4" width="0.1524" layer="91"/>
+<wire x1="60.96" y1="154.94" x2="60.96" y2="152.4" width="0.1524" layer="91"/>
+<junction x="60.96" y="152.4"/>
+<wire x1="50.8" y1="152.4" x2="50.8" y2="144.78" width="0.1524" layer="91"/>
+<junction x="50.8" y="152.4"/>
+<wire x1="50.8" y1="144.78" x2="55.88" y2="144.78" width="0.1524" layer="91"/>
+<label x="55.88" y="144.78" size="1.27" layer="95" xref="yes"/>
 </segment>
 </net>
@@
 <wire x1="193.04" y1="53.34" x2="195.58" y2="53.34" width="0.1524" layer="91"/>
 <label x="195.58" y="53.34" size="1.27" layer="95" font="vector" xref="yes"/>
-</segment>
-</net>
-<net name="N$31" class="0">
-<segment>
-<pinref part="J1" gate="G$1" pin="3"/>
-<pinref part="U1" gate="U1" pin="SCL/D3"/>
-<wire x1="68.58" y1="149.86" x2="45.72" y2="149.86" width="0.1524" layer="91"/>
-<pinref part="R2" gate="G$1" pin="1"/>
-<wire x1="45.72" y1="149.86" x2="40.64" y2="149.86" width="0.1524" layer="91"/>
-<wire x1="45.72" y1="154.94" x2="45.72" y2="149.86" width="0.1524" layer="91"/>
-<junction x="45.72" y="149.86"/>
-</segment>
-</net>
-<net name="N$32" class="0">
-<segment>
-<pinref part="U1" gate="U1" pin="SDA/D2"/>
-<pinref part="J1" gate="G$1" pin="4"/>
-<wire x1="40.64" y1="152.4" x2="60.96" y2="152.4" width="0.1524" layer="91"/>
-<pinref part="R3" gate="G$1" pin="1"/>
-<wire x1="60.96" y1="152.4" x2="68.58" y2="152.4" width="0.1524" layer="91"/>
-<wire x1="60.96" y1="154.94" x2="60.96" y2="152.4" width="0.1524" layer="91"/>
-<junction x="60.96" y="152.4"/>
 </segment>
 </net>
@@
 </segment>
 </net>
-<net name="!RST" class="0">
+<net name="!RST_ATTINY" class="0">
 <segment>
 <pinref part="J2" gate="G$1" pin="5"/>
@@
 </segment>
 </net>
-<net name="INT" class="0">
+<net name="!INT" class="0">
 <segment>
 <pinref part="U5" gate="U1" pin="(ADC7)PA7"/>
@@
 </segment>
 </net>
-<net name="CS" class="0">
+<net name="!CS" class="0">
 <segment>
 <pinref part="J3" gate="G$1" pin="CS"/>
@@
 </segment>
 </net>
-<net name="!RESET" class="0">
+<net name="!RST_SCREEN" class="0">
 <segment>
 <pinref part="J3" gate="G$1" pin="RESET"/>
@@
 </segment>
 </net>
+<net name="N$4" class="0">
+<segment>
+<pinref part="J3" gate="G$1" pin="LEDA"/>
+<wire x1="78.74" y1="104.14" x2="71.12" y2="104.14" width="0.1524" layer="91"/>
+<pinref part="JP1" gate="G$1" pin="1"/>
+<wire x1="71.12" y1="106.68" x2="71.12" y2="104.14" width="0.1524" layer="91"/>
+</segment>
+</net>
+<net name="N$5" class="0">
+<segment>
+<pinref part="U4" gate="G$1" pin="SPEAKER_RN"/>
+<pinref part="J4" gate="G$1" pin="1"/>
+<wire x1="91.44" y1="38.1" x2="88.9" y2="38.1" width="0.1524" layer="91"/>
+</segment>
+</net>
+<net name="N$7" class="0">
+<segment>
+<pinref part="U4" gate="G$1" pin="SPEAKER_RP"/>
+<pinref part="J4" gate="G$1" pin="2"/>
+<wire x1="91.44" y1="40.64" x2="88.9" y2="40.64" width="0.1524" layer="91"/>
+</segment>
+</net>
+<net name="N$10" class="0">
+<segment>
+<pinref part="U4" gate="G$1" pin="MONO_OUT"/>
+<pinref part="TP1" gate="G$1" pin="1"/>
+<wire x1="91.44" y1="45.72" x2="88.9" y2="45.72" width="0.1524" layer="91"/>
+</segment>
+</net>
