File: Hardware/raspi mockup.sch (EAGLE design)
At the start: 51 parts, among them J1 QWIIC, J2 AVR_SPI_PROG_3X2TESTPOINTS, J3 2.4" TFT, U1 RASPBERRY_PI_40BTM-NOHOLES, U2 ADMP401, U3 ADMP401, U4 WM8960, U5 ATTINY84

Commit message: pre design review for REDs
Parts:
- removed J4: (no value), SparkFun-Connectors:CONN_021X02_NO_SILK
- removed TP1: TEST-POINT3X4, SparkFun-Connectors:TEST-POINT3X4
- added C13: 10nF, SparkFun-Capacitors:10NF-0603-50V-10%
- added Q1: 220mA/50V/3.5Ω, SparkFun-DiscreteSemi:MOSFET-NCH-BSS138
- added Y1: 24 MHz, SparkFun-Clocks:OSCILLATOR-24MHZ
Connections:
- removed net ADC-LRC: U4.ADCLRC/GPIO
- removed net N$10: TP1.1, U4.MONO_OUT
- removed net N$5: J4.1, U4.SPEAKER_RN
- removed net N$7: J4.2, U4.SPEAKER_RP
- new net N$11: U4.MCLK, Y1.OUT
- net 3.3V: now also C13.1, Y1.EN, Y1.VCC
- net DAC-LRC: now also U4.ADCLRC/GPIO
- net GND: now also C13.2, Y1.GND
- net SCL: now also J1.4; no longer J1.3
- net SDA: now also J1.3; no longer J1.4
