File: Hardware/Top pHAT.sch (EAGLE design)
At the start: 51 parts, among them J1 QWIIC, J2 AVR_SPI_PROG_3X2TESTPOINTS, J3 2.4" TFT, U1 RASPBERRY_PI_40BTM-NOHOLES, U2 ADMP401, U3 ADMP401, U4 WM8960, U5 ATTINY84

Commit message: pre design review for REDs
Parts:
- removed J4: (no value), SparkFun-Connectors:CONN_021X02_NO_SILK
- removed JP1: JUMPER-SMT_2_NC_TRACE_NO-SILK, SparkFun-Jumpers:JUMPER-SMT_2_NC_TRACE_NO-SILK
- added C13: 10nF, SparkFun-Capacitors:10NF-0603-50V-10%
- added Q2: 1.1A/60V/600mΩ, SparkFun-DiscreteSemi:MOSFET_PCH-SI2309DS
- added TP10, TP11, TP12, TP13, TP14, TP15, TP2, TP3, TP4, TP5, TP6, TP7, TP8, TP9: TEST-POINT3X5, SparkFun-Connectors:TEST-POINT3X5
- added Y1: 24 MHz, SparkFun-Clocks:OSCILLATOR-24MHZ
- FRAME1: value FRAME-LETTER -> FRAME-LEDGER; device SparkFun-Aesthetics:FRAME-LETTER -> SparkFun-Aesthetics:FRAME-LEDGER
- TP1: value TEST-POINT3X4 -> TEST-POINT3X5; device SparkFun-Connectors:TEST-POINT3X4 -> SparkFun-Connectors:TEST-POINT3X5
Connections:
- removed net ADC-LRC: U4.ADCLRC/GPIO
- removed net N$10: TP1.1, U4.MONO_OUT
- removed net N$5: J4.1, U4.SPEAKER_RN
- removed net N$7: J4.2, U4.SPEAKER_RP
- new net !BKLITE: Q2.G, TP12.1, U1.D22
- new net N$11: U4.MCLK, Y1.OUT
- net !CS: now also TP6.1
- net !INT: now also TP15.1
- net !RST_SCREEN: now also TP13.1
- net 3.3V: now also C13.1, Q2.S, Y1.EN, Y1.VCC; no longer JP1.2
- net ADC-DAT: now also TP10.1
- net BCLK: now also TP8.1
- net D/C: now also TP14.1
- net DAC-DAT: now also TP11.1
- net DAC-LRC: now also TP9.1, U4.ADCLRC/GPIO
- net GND: now also C13.2, Y1.GND
- net LED_DATA: now also TP7.1
- net N$4: now also Q2.D; no longer JP1.1
- net SCK: now also TP5.1
- net SCL: now also J1.4, TP1.1; no longer J1.3
- net SDA: now also J1.3, TP2.1; no longer J1.4
- net SDI: now also TP3.1
- net SDO: now also TP4.1
Other:
- note added: "7-bit Unshifted I2C Address: 0x6F"
- note added: "Test Points"
- note added: "v10"
- note removed: "7-bit Unshifted I2C Address: 0x34"
- note removed: "v01"
- moved on the sheet: C1, C10, C11, C12, C2, C3, C4, C5, C6, C7, C8, C9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

Commit message: post design review
Other:
- moved on the sheet: J3, Q2, R4
Changed lines of the file:
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@@
 <?xml version="1.0" encoding="utf-8"?>
 <!DOCTYPE eagle SYSTEM "eagle.dtd">
-<eagle version="9.5.2">
+<eagle version="9.3.1">
 <drawing>
 <settings>
@@
 <plain>
 <text x="348.742" y="11.43" size="2.54" layer="94" font="vector">Andy England</text>
-<text x="71.12" y="198.12" size="2.54" layer="97" font="vector">Screen</text>
+<text x="165.1" y="187.96" size="2.54" layer="97" font="vector">Screen</text>
 <text x="2.54" y="274.32" size="2.54" layer="97" font="vector">40-Pin Raspberry Pi Connector</text>
 <text x="2.54" y="109.22" size="2.54" layer="97" font="vector">Audio Codec</text>
@@
 <attribute name="VALUE" x="137.16" y="48.006" size="1.27" layer="96" font="vector" rot="R180"/>
 </instance>
-<instance part="J3" gate="G$1" x="109.22" y="175.26" smashed="yes">
-<attribute name="NAME" x="99.06" y="185.928" size="1.778" layer="95" font="vector"/>
-<attribute name="VALUE" x="99.06" y="165.1" size="1.778" layer="96" font="vector"/>
-</instance>
-<instance part="SUPPLY11" gate="G$1" x="93.98" y="193.04" smashed="yes" rot="MR0">
-<attribute name="VALUE" x="93.98" y="195.834" size="1.778" layer="96" rot="MR0" align="bottom-center"/>
-</instance>
-<instance part="GND9" gate="1" x="91.44" y="165.1" smashed="yes" rot="MR0">
-<attribute name="VALUE" x="91.44" y="164.846" size="1.778" layer="96" rot="MR0" align="top-center"/>
+<instance part="J3" gate="G$1" x="223.52" y="147.32" smashed="yes">
+<attribute name="NAME" x="213.36" y="157.988" size="1.778" layer="95" font="vector"/>
+<attribute name="VALUE" x="213.36" y="137.16" size="1.778" layer="96" font="vector"/>
+</instance>
+<instance part="SUPPLY11" gate="G$1" x="208.28" y="165.1" smashed="yes" rot="MR0">
+<attribute name="VALUE" x="208.28" y="167.894" size="1.778" layer="96" rot="MR0" align="bottom-center"/>
+</instance>
+<instance part="GND9" gate="1" x="205.74" y="137.16" smashed="yes" rot="MR0">
+<attribute name="VALUE" x="205.74" y="136.906" size="1.778" layer="96" rot="MR0" align="top-center"/>
 </instance>
 <instance part="LOGO1" gate="G$1" x="205.74" y="7.62" smashed="yes"/>
@@
 <instance part="FD3" gate="G$1" x="421.64" y="17.78" smashed="yes"/>
 <instance part="FD4" gate="G$1" x="424.18" y="17.78" smashed="yes"/>
-<instance part="R4" gate="G$1" x="139.7" y="185.42" smashed="yes" rot="R90">
-<attribute name="NAME" x="138.176" y="185.42" size="1.778" layer="95" font="vector" rot="R90" align="bottom-center"/>
-<attribute name="VALUE" x="141.224" y="185.42" size="1.778" layer="96" font="vector" rot="R90" align="top-center"/>
-</instance>
-<instance part="SUPPLY12" gate="G$1" x="139.7" y="193.04" smashed="yes" rot="MR0">
-<attribute name="VALUE" x="139.7" y="195.834" size="1.778" layer="96" rot="MR0" align="bottom-center"/>
+<instance part="R4" gate="G$1" x="254" y="157.48" smashed="yes" rot="R90">
+<attribute name="NAME" x="252.476" y="157.48" size="1.778" layer="95" font="vector" rot="R90" align="bottom-center"/>
+<attribute name="VALUE" x="255.524" y="157.48" size="1.778" layer="96" font="vector" rot="R90" align="top-center"/>
+</instance>
+<instance part="SUPPLY12" gate="G$1" x="254" y="165.1" smashed="yes" rot="MR0">
+<attribute name="VALUE" x="254" y="167.894" size="1.778" layer="96" rot="MR0" align="bottom-center"/>
 </instance>
 <instance part="Y1" gate="G$1" x="45.72" y="33.02" smashed="yes">
@@
 <attribute name="VALUE" x="25.4" y="22.606" size="1.778" layer="96" align="top-center"/>
 </instance>
-<instance part="Q2" gate="G$1" x="86.36" y="182.88" smashed="yes" rot="MR180">
-<attribute name="NAME" x="83.82" y="187.96" size="1.778" layer="95" font="vector" rot="MR180"/>
-<attribute name="VALUE" x="81.28" y="162.56" size="1.778" layer="96" font="vector" rot="MR90"/>
+<instance part="Q2" gate="G$1" x="200.66" y="154.94" smashed="yes" rot="MR180">
+<attribute name="NAME" x="198.12" y="160.02" size="1.778" layer="95" font="vector" rot="MR180"/>
+<attribute name="VALUE" x="195.58" y="134.62" size="1.778" layer="96" font="vector" rot="MR90"/>
 </instance>
 <instance part="FRAME1" gate="G$1" x="0" y="0" smashed="yes"/>
@@
 <segment>
 <pinref part="SUPPLY11" gate="G$1" pin="3.3V"/>
-<wire x1="93.98" y1="193.04" x2="93.98" y2="190.5" width="0.1524" layer="91"/>
+<wire x1="208.28" y1="165.1" x2="208.28" y2="162.56" width="0.1524" layer="91"/>
 <pinref part="J3" gate="G$1" pin="VCC"/>
-<wire x1="93.98" y1="190.5" x2="93.98" y2="182.88" width="0.1524" layer="91"/>
-<wire x1="93.98" y1="182.88" x2="96.52" y2="182.88" width="0.1524" layer="91"/>
-<wire x1="93.98" y1="190.5" x2="88.9" y2="190.5" width="0.1524" layer="91"/>
-<junction x="93.98" y="190.5"/>
+<wire x1="208.28" y1="162.56" x2="208.28" y2="154.94" width="0.1524" layer="91"/>
+<wire x1="208.28" y1="154.94" x2="210.82" y2="154.94" width="0.1524" layer="91"/>
+<wire x1="208.28" y1="162.56" x2="203.2" y2="162.56" width="0.1524" layer="91"/>
+<junction x="208.28" y="162.56"/>
 <pinref part="Q2" gate="G$1" pin="S"/>
-<wire x1="88.9" y1="187.96" x2="88.9" y2="190.5" width="0.1524" layer="91"/>
+<wire x1="203.2" y1="160.02" x2="203.2" y2="162.56" width="0.1524" layer="91"/>
 </segment>
 <segment>
 <pinref part="SUPPLY12" gate="G$1" pin="3.3V"/>
 <pinref part="R4" gate="G$1" pin="2"/>
-<wire x1="139.7" y1="193.04" x2="139.7" y2="190.5" width="0.1524" layer="91"/>
+<wire x1="254" y1="165.1" x2="254" y2="162.56" width="0.1524" layer="91"/>
 </segment>
 </net>
@@
 <segment>
 <pinref part="J3" gate="G$1" pin="LEDK"/>
-<wire x1="96.52" y1="177.8" x2="91.44" y2="177.8" width="0.1524" layer="91"/>
+<wire x1="210.82" y1="149.86" x2="205.74" y2="149.86" width="0.1524" layer="91"/>
 <pinref part="J3" gate="G$1" pin="GND"/>
-<wire x1="91.44" y1="177.8" x2="91.44" y2="170.18" width="0.1524" layer="91"/>
-<wire x1="91.44" y1="170.18" x2="96.52" y2="170.18" width="0.1524" layer="91"/>
-<wire x1="91.44" y1="170.18" x2="91.44" y2="167.64" width="0.1524" layer="91"/>
-<junction x="91.44" y="170.18"/>
+<wire x1="205.74" y1="149.86" x2="205.74" y2="142.24" width="0.1524" layer="91"/>
+<wire x1="205.74" y1="142.24" x2="210.82" y2="142.24" width="0.1524" layer="91"/>
+<wire x1="205.74" y1="142.24" x2="205.74" y2="139.7" width="0.1524" layer="91"/>
+<junction x="205.74" y="142.24"/>
 <pinref part="GND9" gate="1" pin="GND"/>
 </segment>
@@
 <segment>
 <pinref part="J3" gate="G$1" pin="SCK"/>
-<wire x1="121.92" y1="177.8" x2="124.46" y2="177.8" width="0.1524" layer="91"/>
-<label x="124.46" y="177.8" size="1.27" layer="95" xref="yes"/>
+<wire x1="236.22" y1="149.86" x2="238.76" y2="149.86" width="0.1524" layer="91"/>
+<label x="238.76" y="149.86" size="1.27" layer="95" xref="yes"/>
 </segment>
 <segment>
@@
 <segment>
 <pinref part="J3" gate="G$1" pin="CS"/>
-<wire x1="121.92" y1="175.26" x2="139.7" y2="175.26" width="0.1524" layer="91"/>
-<label x="139.7" y="172.72" size="1.27" layer="95" xref="yes"/>
+<wire x1="236.22" y1="147.32" x2="254" y2="147.32" width="0.1524" layer="91"/>
+<label x="254" y="144.78" size="1.27" layer="95" xref="yes"/>
 <pinref part="R4" gate="G$1" pin="1"/>
-<wire x1="139.7" y1="175.26" x2="139.7" y2="172.72" width="0.1524" layer="91"/>
-<wire x1="139.7" y1="180.34" x2="139.7" y2="175.26" width="0.1524" layer="91"/>
-<junction x="139.7" y="175.26"/>
+<wire x1="254" y1="147.32" x2="254" y2="144.78" width="0.1524" layer="91"/>
+<wire x1="254" y1="152.4" x2="254" y2="147.32" width="0.1524" layer="91"/>
+<junction x="254" y="147.32"/>
 </segment>
 <segment>
@@
 <segment>
 <pinref part="J3" gate="G$1" pin="D/C"/>
-<wire x1="121.92" y1="172.72" x2="124.46" y2="172.72" width="0.1524" layer="91"/>
-<label x="124.46" y="172.72" size="1.27" layer="95" xref="yes"/>
+<wire x1="236.22" y1="144.78" x2="238.76" y2="144.78" width="0.1524" layer="91"/>
+<label x="238.76" y="144.78" size="1.27" layer="95" xref="yes"/>
 </segment>
 <segment>
@@
 <segment>
 <pinref part="J3" gate="G$1" pin="SDI"/>
-<wire x1="121.92" y1="182.88" x2="124.46" y2="182.88" width="0.1524" layer="91"/>
-<label x="124.46" y="182.88" size="1.27" layer="95" xref="yes"/>
+<wire x1="236.22" y1="154.94" x2="238.76" y2="154.94" width="0.1524" layer="91"/>
+<label x="238.76" y="154.94" size="1.27" layer="95" xref="yes"/>
 </segment>
 <segment>
@@
 <segment>
 <pinref part="J3" gate="G$1" pin="SDO"/>
-<wire x1="121.92" y1="170.18" x2="124.46" y2="170.18" width="0.1524" layer="91"/>
-<label x="124.46" y="170.18" size="1.27" layer="95" xref="yes"/>
+<wire x1="236.22" y1="142.24" x2="238.76" y2="142.24" width="0.1524" layer="91"/>
+<label x="238.76" y="142.24" size="1.27" layer="95" xref="yes"/>
 </segment>
 <segment>
@@
 <segment>
 <pinref part="J3" gate="G$1" pin="RESET"/>
-<wire x1="121.92" y1="180.34" x2="124.46" y2="180.34" width="0.1524" layer="91"/>
-<label x="124.46" y="180.34" size="1.27" layer="95" xref="yes"/>
+<wire x1="236.22" y1="152.4" x2="238.76" y2="152.4" width="0.1524" layer="91"/>
+<label x="238.76" y="152.4" size="1.27" layer="95" xref="yes"/>
 </segment>
 <segment>
@@
 <segment>
 <pinref part="J3" gate="G$1" pin="LEDA"/>
-<wire x1="96.52" y1="175.26" x2="88.9" y2="175.26" width="0.1524" layer="91"/>
-<wire x1="88.9" y1="177.8" x2="88.9" y2="175.26" width="0.1524" layer="91"/>
+<wire x1="210.82" y1="147.32" x2="203.2" y2="147.32" width="0.1524" layer="91"/>
+<wire x1="203.2" y1="149.86" x2="203.2" y2="147.32" width="0.1524" layer="91"/>
 <pinref part="Q2" gate="G$1" pin="D"/>
 </segment>
@@
 <segment>
 <pinref part="Q2" gate="G$1" pin="G"/>
-<wire x1="81.28" y1="185.42" x2="78.74" y2="185.42" width="0.1524" layer="91"/>
-<label x="78.74" y="185.42" size="1.27" layer="95" rot="R180" xref="yes"/>
-</segment>
-<segment>
+<wire x1="195.58" y1="157.48" x2="193.04" y2="157.48" width="0.1524" layer="91"/>
+<label x="193.04" y="157.48" size="1.27" layer="95" rot="R180" xref="yes"/>
+</segment>
+<segment>
